File: ems.sch (KiCad schematic (older format))
At the start: 88 parts, among them J1 Conn_01x15, U1 LTC2983, U2 TL071, U3 TL071

Commit message: Updated schematic
Parts:
- removed U2, U3: TL071, symbol TL071
- added U2: LM324, symbol LM324
Connections:
- net FUEL-FLOW: now also U2.7
- net GND: now also U2.11 (V-), U2.11 (V-)
- net HALL: now also U2.1
- net VDD: now also U2.4 (V+), U2.4 (V+)
- net at RV6.2: now also U2.2 (-)
- net at C26.2, R21.2, R22.2: now also U2.3 (+)
- net at RV8.2: now also U2.6 (-)
- net at C28.2, R27.2, R31.2: now also U2.5 (+)
Changed lines of the file:
@@
-$EndComp
-$Comp
-L TL071 U2
-U 1 1 5B27F35B
-P 9600 5600
-F 0 "U2" H 9600 5850 50  0000 L CNN
-F 1 "TL071" H 9600 5750 50  0000 L CNN
-F 2 "" H 9650 5650 50  0001 C CNN
-F 3 "" H 9750 5750 50  0001 C CNN
-	1    9600 5600
-	1    0    0    -1
 $EndComp
 $Comp
@@
 Wire Wire Line
 	4450 3650 5100 3650
-$Comp
-L TL071 U3
-U 1 1 5B292A0D
-P 12100 5700
-F 0 "U3" H 12100 5950 50  0000 L CNN
-F 1 "TL071" H 12100 5850 50  0000 L CNN
-F 2 "" H 12150 5750 50  0001 C CNN
-F 3 "" H 12250 5850 50  0001 C CNN
-	1    12100 5700
-	1    0    0    -1
-$EndComp
 $Comp
 L POT RV8
@@
 Wire Wire Line
 	7200 3150 7350 3150
+$Comp
+L LM324 U2
+U 1 1 5B6A7EFF
+P 9600 5600
+F 0 "U2" H 9600 5800 50  0000 L CNN
+F 1 "LM324" H 9600 5400 50  0000 L CNN
+F 2 "" H 9550 5700 50  0001 C CNN
+F 3 "" H 9650 5800 50  0001 C CNN
+	1    9600 5600
+	1    0    0    -1
+$EndComp
+$Comp
+L LM324 U2
+U 2 1 5B6A984D
+P 12100 5700
+F 0 "U2" H 12100 5900 50  0000 L CNN
+F 1 "LM324" H 12100 5500 50  0000 L CNN
+F 2 "" H 12050 5800 50  0001 C CNN
+F 3 "" H 12150 5900 50  0001 C CNN
+	2    12100 5700
+	1    0    0    -1
+$EndComp
+Wire Wire Line
+	12750 5150 12475 5150
+Wire Wire Line
+	12475 5150 12475 5400
+Wire Wire Line
+	12475 5400 12000 5400
+Wire Wire Line
+	11500 6250 12000 6250
+Wire Wire Line
+	12000 6250 12000 6000
+Wire Wire Line
+	10250 5050 10025 5050
+Wire Wire Line
+	10025 5050 10025 5300
+Wire Wire Line
+	10025 5300 9500 5300
+Wire Wire Line
+	9500 5900 9500 6150
+Wire Wire Line
+	9500 6150 9000 6150
 $EndSCHEMATC
